Commit message: - 두산 로봇 lerobot 데이터 수집 및 인퍼런스 기능 추가

File: ik_solver/contents/dsr-m1013.urdf (robot description, URDF)
Before this commit: robot dsr-m1013, 8 links, 7 joints
Links:
- added link end_effector, mass 1; collision box size=0.1 0.1 0.1; visual box size=0.1 0.1 0.1
- added link flange, mass 1; collision box size=0.1 0.1 0.1; visual box size=0.1 0.1 0.1
- link base: mass None -> 1; geometry visual box size=0.1 0.1 0.1
- link base_0: geometry visual box size=0.1 0.1 0.1
- link link1: geometry collision box size=0.1 0.1 0.1; visual box size=0.1 0.1 0.1
- link link2: geometry collision box size=0.1 0.1 0; visual box size=0.1 0.1 0.1
- link link3: geometry collision box size=0.1 0.1 0.1; visual box size=0.1 0.1 0.1
- link link4: geometry collision box size=0.1 0.1 0.1; visual box size=0.1 0.1 0.1
- link link5: geometry collision box size=0.1 0.1 0.1; visual box size=0.1 0.1 0.1
- link link6: geometry collision box size=0.1 0.1 0.1; visual box size=0.1 0.1 0.1
Joints:
- added joint end_effector: type fixed, parent flange, child end_effector, origin xyz=0 0 0 rpy=0 0 0, axis 0 0 1
- added joint flange: type fixed, parent link6, child flange, origin xyz=0 0 0 rpy=0 0 0, axis 0 0 1
